File: atmega328P.sch (KiCad schematic (older format))
At the start: 26 parts, among them IC3 ATMEGA328P-AU, IC4 FT232RL-REEL, Y2 16 MHz

Commit message: hub schematic finished
Parts:
- removed C10, C12: 0.1 uF, SamacSys_Parts:CAPC3216X88N, symbol SamacSys_Parts:C1206C104K5RAC7411
- removed C11, C28, C29, C30: 0,1 uF, SamacSys_Parts:CAPC3216X88N, symbol SamacSys_Parts:C1206C104K5RAC7411
- removed C31, C32, C33, C34, C35: 1 uF, SamacSys_Parts:CAPC3216X210N, symbol SamacSys_Parts:SH31B105K500CT
- removed C8, C9: 22 pF, SamacSys_Parts:CAPC2012X70N, symbol SamacSys_Parts:885012007002
- removed IC3: ATMEGA328P-AU, SamacSys_Parts:QFP80P900X900X120-32N, symbol SamacSys_Parts:ATMEGA328P-AU
- removed IC4: FT232RL-REEL, SamacSys_Parts:SOP65P778X200-28N, symbol SamacSys_Parts:FT232RL-REEL
- removed LED1, LED2, LED3: Green, SamacSys_Parts:LEDC3214X78N, symbol SamacSys_Parts:150120GS75000
- removed R24, R26, R28, R29, R30: 1 K, SamacSys_Parts:RESC3216X60N, symbol SamacSys_Parts:CRCW12061K00JNEAHP
- removed R25: 240 R, SamacSys_Parts:RESC3216X75N, symbol SamacSys_Parts:CR1206-FX-2400ELF
- removed R27: 10 K, SamacSys_Parts:RESC3216X60N, symbol SamacSys_Parts:CRCW120610K0FKEAC
- removed Y2: 16 MHz, SamacSys_Parts:ECS49205PXTR, symbol SamacSys_Parts:ECS-160-18-5PX-JES-TR
