File: atmega32.kicad_pcb (KiCad board)
At the start: 4 copper layers, 74.7 x 62.2 mm, 26 parts, among them J1 USB_B_Micro, J2 20021111-00016T4LF, U1 ATmega328P-AU, U2 FT232RL

Commit message: finished eval board
Parts:
- added C10: 4.7uF, storage:C_4.7uF, F.Cu at (121.9, 127.0)
- added C11: 0.1u, storage:C_0.1uF, F.Cu at (105.8, 116.1)
- added C12: 0.1u, storage:C_0.1uF, F.Cu at (105.8, 118.4)
- added C13: 0.1u, storage:C_0.1uF, F.Cu at (122.2, 121.2)
- added C7: 0.1u, storage:C_0.1uF, F.Cu at (150.6, 112.0)
- added C8: 22pF, storage:C_0.1uF, F.Cu at (107.2, 134.8)
- added C9: 22pF, storage:C_0.1uF, F.Cu at (106.8, 121.9)
- added D4: SCK, storage:LED_WL-SMCW, F.Cu at (119.8, 132.5)
- added G***: LOGO, logo_arduino:logo, F.Cu at (144.5, 144.8)
- added R10: 1K, storage:R_1K, F.Cu at (120.1, 135.5)
- added R9: 1K, storage:R_1K, F.Cu at (146.7, 109.0)
- added SW1: SW_MEC_5E, storage:Button, F.Cu at (149.9, 99.1)
- added Y1: Crystal, SamacSys_Parts:ECS49205PXTR, F.Cu at (102.6, 130.7)
- moved C1 44.0 mm to (131.6, 138.4)
- moved C2 44.0 mm to (139.3, 138.4), turned to 180 degrees
- moved U1 36.9 mm to (114.1, 120.8), turned to 0 degrees
- moved R5 36.6 mm to (136.7, 137.0), turned to 270 degrees
- moved C5 35.4 mm to (145.4, 112.2), turned to 270 degrees
- moved R7 32.5 mm to (114.3, 110.0), turned to 180 degrees
- moved R8 32.3 mm to (113.0, 112.5), turned to 180 degrees
- moved R1 31.9 mm to (157.0, 126.2)
- moved D1 31.2 mm to (161.9, 126.2), turned to 0 degrees
- moved R2 31.0 mm to (157.0, 129.4)
- moved D2 29.5 mm to (161.9, 129.3)
- moved U2 24.0 mm to (143.2, 120.4), turned to 270 degrees
- moved C6 22.7 mm to (141.1, 134.7), turned to 180 degrees
- moved F1 17.9 mm to (129.0, 145.0), turned to 0 degrees
- moved C4 16.7 mm to (142.5, 127.9)
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Connections:
- C1 pad 1: D- -> GND
- C2 pad 1: D- -> GND
- C3 pad 1: D- -> GND
- C3 pad 2: VBUS -> +5V
- C4 pad 1: VBUS -> +5V
- C4 pad 2: D- -> GND
- C5 pad 1: D- -> GND
- C5 pad 2: VBUS -> +5V
- C6 pad 1: D- -> GND
- F1 pad 1: VBUS -> +5V
- H1 pad 1: D- -> GND
- H2 pad 1: D- -> GND
- H3 pad 1: D- -> GND
- H4 pad 1: D- -> GND
- J1 pad 5: D- -> GND
- J2 pad 1: (no net) -> /MISO
- J2 pad 10: (no net) -> /ADC7
- J2 pad 11: (no net) -> /PD4
- J2 pad 12: (no net) -> /PD6
- J2 pad 13: (no net) -> /PC4
- J2 pad 14: (no net) -> /PC5
- J2 pad 15: D- -> GND
- J2 pad 2: (no net) -> +5V
- J2 pad 3: (no net) -> /SCK
- J2 pad 4: (no net) -> /MOSI
- J2 pad 5: (no net) -> /RESET
- J2 pad 6: (no net) -> GND
- J2 pad 7: (no net) -> /INT0
- J2 pad 8: (no net) -> /INT1
- J2 pad 9: (no net) -> /ADC6
- R3 pad 2: D- -> GND
- R6 pad 2: D- -> GND
- U1 pad 1: (no net) -> /INT1
- U1 pad 10: (no net) -> /PD6
- U1 pad 15: (no net) -> /MOSI
- U1 pad 16: (no net) -> /MISO
- U1 pad 17: (no net) -> /SCK
- U1 pad 18: (no net) -> +5V
- U1 pad 19: (no net) -> /ADC6
- U1 pad 2: (no net) -> /PD4
- U1 pad 20: (no net) -> Net-(C13-Pad1)
- U1 pad 21: Net-(U1-Pad21) -> GND
- U1 pad 22: (no net) -> /ADC7
- U1 pad 27: (no net) -> /PC4
- U1 pad 28: (no net) -> /PC5
- U1 pad 29: (no net) -> /RESET
- U1 pad 3: Net-(U1-Pad21) -> GND
- U1 pad 32: (no net) -> /INT0
- U1 pad 4: Net-(U1-Pad4) -> +5V
- U1 pad 5: Net-(U1-Pad21) -> GND
- U1 pad 6: Net-(U1-Pad4) -> +5V
- U1 pad 7: (no net) -> /XTAL1
- U1 pad 8: (no net) -> /XTAL2
- U2 pad 18: D- -> GND
- U2 pad 2: (no net) -> DTR
- U2 pad 20: VBUS -> +5V
- U2 pad 21: D- -> GND
- U2 pad 25: D- -> GND
- U2 pad 26: D- -> GND
- U2 pad 4: VBUS -> +5V
- U2 pad 7: D- -> GND
Routing:
- net /RESET: track 0.00 -> 80.1 mm, vias 0 -> 4
- net /SCK: track 0.00 -> 71.0 mm, vias 0 -> 3
- net +3V3: track 0.00 -> 66.4 mm, vias 0 -> 1
- net /MISO: track 0.00 -> 64.1 mm, vias 0 -> 3
- net GND: track 0.00 -> 62.2 mm, vias 0 -> 25
- net /MOSI: track 0.00 -> 56.8 mm, vias 0 -> 1
- net /PD6: track 0.00 -> 45.7 mm, vias 0 -> 5
- net /INT1: track 0.00 -> 40.5 mm, vias 0 -> 4
- net TXD: track 0.00 -> 37.2 mm
- net /ADC7: track 0.00 -> 35.8 mm, vias 0 -> 3
- net RXD: track 0.00 -> 35.3 mm, vias 0 -> 2
- net /INT0: track 0.00 -> 34.8 mm, vias 0 -> 1
- net /PC5: track 0.00 -> 34.2 mm, vias 0 -> 3
- net /PD4: track 0.00 -> 32.5 mm, vias 0 -> 2
- net +5V: track 0.00 -> 31.6 mm, vias 0 -> 11
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- added copper zone on F.Cu, net +5V
- added copper zone on In2.Cu, net +5V
- added copper zone on F.Cu, net GND
- added copper zone on In1.Cu, net GND
Other:
- board text added: "Atmega32 Evalboard by Maximilian Altrichter"
