File: atmega32.sch (KiCad schematic (older format))
At the start: 29 parts, among them J1 USB_B_Micro, J2 20021111-00016T4LF, SW1 SW_MEC_5G, U1 ATmega328P-AU, U2 FT232RL

Commit message: finished eval board
Parts:
- removed SW1: SW_MEC_5G, symbol Switch:SW_MEC_5G
- added C10: 4.7uF, storage:C_4.7uF, symbol Device:CP_Small
- added C11, C12, C13: 0.1u, storage:C_0.1uF, symbol Device:C_Small
- added C8, C9: 22pF, storage:C_0.1uF, symbol Device:C_Small
- added D4: SCK, storage:LED_WL-SMCW, symbol Device:LED_Small
- added R10: 1K, storage:R_1K, symbol Device:R_Small
- added SW1: SW_MEC_5E, storage:Button, symbol Switch:SW_MEC_5E
- added Y1: Crystal, SamacSys_Parts:ECS49205PXTR, symbol Device:Crystal
Connections:
- net labels added: ADC6, ADC7, INT0, INT1, MISO, MOSI, PC4, PC5, PD4, PD6, SCK, XTAL1, XTAL2
- net labels removed: VBUS
- wire segments 90 -> 139
- no-connect marks 11 -> 21
Other:
- note added: "Crystal"
- moved on the sheet: R7, R8, U1

Commit message: orderd
Other:
- note added: "Atmega32"
- moved on the sheet: C10, C11, C12, C13, D4, R10, R7, R8, U1
