File: sh_control.kicad_pcb (KiCad board)
At the start: 4 copper layers, 86.4 x 94.7 mm, 90 parts, among them IC1 SN75240PW, IC2 LM317MDCY, IC3 TPS73533DRBT, IC4 TLV76733DGNR, IC5 TUSB2046IBVF, IC6 TPS2044BDR, IC7 SN75240PW, J1 USB_B_Micro, J2 10129381-906001BLF, J3 10129381-906001BLF, SW1 Reset, Y1 6MHz

Commit message: start V3.3
Parts:
- removed Buck_1: Buck_1, SamacSys_Parts:LEDC3214X78N
- removed Buck_2: Buck_2, SamacSys_Parts:LEDC3214X78N
- removed C10: 2.2uF, storage:C_2.2F
- removed C11, C13, C14, C6: 0.1uF, storage:C_0.1uF
- removed C12, C17, C18: 4.7uF, storage:C_4.7uF
- removed C15, C16, C21, C22, C23, C24, C27, C28, C29, C30, C5, C7: 22pF, storage:C_22pF
- removed C19, C20: 27uF, storage:C_27pF
- removed C25, C26, C31, C32: 100uF, storage:C_100uF
- removed C8, C9: 1uF, storage:C_1uF
- removed Enable1: TestPoint, TestPoint:TestPoint_Pad_D2.5mm
- removed GND1: GND, TestPoint:TestPoint_Pad_D2.5mm
- removed IC3: TPS73533DRBT, SamacSys_Parts:TPS73533DRBT
- removed IC4: TLV76733DGNR, SamacSys_Parts:SOP65P490X110-9N
- removed IC5: TUSB2046IBVF, SamacSys_Parts:QFP80P900X900X160-32N
- removed IC6: TPS2044BDR, SamacSys_Parts:SOIC127P600X175-16N
- removed IC7: SN75240PW, SamacSys_Parts:SOP65P640X120-8N
- removed LDO1: LDO, SamacSys_Parts:LEDC3214X78N
- removed PortA1, PortB1, PortC1, PortD1: USB_A, Connector_USB:USB_A_Molex_67643_Horizontal
- removed R10, R18, R6: 1.5k, storage:R_1K5
- removed R11, R12, R13: 1k, storage:R_1K
- removed R14, R15, R16, R17, R19, R20, R21, R22, R4, R5: 22, storage:R_22
- removed R23, R24, R25, R26, R27, R28, R29, R30: 15k, storage:R_15K
- removed R7: 240, storage:R_240
- removed R8: 390, storage:R_390
- removed R9: 10k, storage:R_10K
- removed SW1: Reset, SamacSys_Parts:FSM4JH
- removed VBUS1: VBUS, TestPoint:TestPoint_Pad_D2.5mm
- removed Y1: 6MHz, SamacSys_Parts:LFXTAL036567BULK
- added J4: 692121030100, SamacSys_Parts:692121030100, F.Cu at (85.6, 68.9)
- added J5: 692121030100, SamacSys_Parts:692121030100, F.Cu at (103.3, 68.9)
- C2: value 1uF -> 10uF; footprint storage:C_1uF -> storage:C_10uF
- C3: value 1uF -> 0.1uF; footprint storage:C_1uF -> storage:C_0.1uF
- C4: value 10uF -> 0.1uF; footprint storage:C_10uF -> storage:C_0.1uF
- IC1: value SN75240PW -> LM317MDCY; footprint SamacSys_Parts:SOP65P640X120-8N -> SamacSys_Parts:SOT230P700X180-4N
- IC2: value LM317MDCY -> TUSB8041IPAPRQ1; footprint SamacSys_Parts:SOT230P700X180-4N -> SamacSys_Parts:QFP50P1200X1200X120-65N
- J1: value USB_B_Micro -> 692221030100; footprint Connector_USB:USB_Micro-B_Molex-105017-0001 -> SamacSys_Parts:WR-COM_USB_TYPE_B
- J2, J3: value 10129381-906001BLF -> 692121030100; footprint SamacSys_Parts:HDRV6W67P254_2X3_762X483X858P -> SamacSys_Parts:692121030100
- R2: value 390 -> 240; footprint storage:R_390 -> storage:R_240
- R3: value 22 -> 390; footprint storage:R_22 -> storage:R_390
- moved R2 138.0 mm to (66.6, 123.3)
- moved C1 131.2 mm to (76.6, 128.5)
- moved D1 126.0 mm to (65.3, 115.4), turned to 0 degrees
- moved H2 123.8 mm to (30.5, 127.0)
- moved IC2 118.9 mm to (47.2, 99.4)
- moved J3 112.1 mm to (50.4, 68.9), turned to 180 degrees
- moved D2 106.6 mm to (65.3, 119.5)
- moved H4 99.4 mm to (30.5, 73.7)
- moved C3 98.4 mm to (83.2, 123.2), turned to 0 degrees
- moved C4 96.7 mm to (87.1, 128.3), turned to 0 degrees
- moved C2 96.4 mm to (82.0, 128.3), turned to 0 degrees
- moved H3 91.0 mm to (109.2, 73.7)
- moved R3 85.8 mm to (72.2, 123.3), turned to 0 degrees
- moved H1 83.9 mm to (109.2, 127.0)
- moved IC1 77.7 mm to (85.7, 117.5)
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Connections:
- C1 pad 1: LDO -> Net-(C1-Pad1)
- C2 pad 1: Buck_1 -> Net-(C2-Pad1)
- C3 pad 1: 3V3_Buck_2 -> Net-(C2-Pad1)
- C4 pad 1: Buck_2 -> Net-(C4-Pad1)
- D1 pad 1: Net-(C13-Pad1) -> Net-(C4-Pad1)
- D1 pad 2: 3V3_Buck_2 -> Net-(C1-Pad1)
- D2 pad 1: Buck_2 -> Net-(C2-Pad1)
- D2 pad 2: Net-(C13-Pad1) -> Net-(C4-Pad1)
- IC1 pad 1: GND -> Net-(IC1-Pad1)
- IC1 pad 2: Net-(IC1-Pad2) -> Net-(C1-Pad1)
- IC1 pad 3: GND -> Net-(C2-Pad1)
- IC1 pad 4: Net-(IC1-Pad4) -> Net-(C4-Pad1)
- IC2 pad 1: Net-(IC2-Pad1) -> (no net)
- IC2 pad 2: 3V3_Buck_2 -> (no net)
- IC2 pad 3: Buck_2 -> (no net)
- IC2 pad 4: Net-(C13-Pad1) -> (no net)
- J1 pad 1: VBUS -> (no net)
- J1 pad 2: Net-(IC1-Pad4) -> (no net)
- J1 pad 3: Net-(IC1-Pad2) -> (no net)
- J1 pad 5: GND -> (no net)
- J1 pad 6: Net-(J1-Pad6) -> (no net)
- J2 pad 1: VBUS -> (no net)
- J2 pad 2: Buck_1 -> (no net)
- J2 pad 3: VBUS -> (no net)
- J2 pad 4: Buck_2 -> (no net)
- J2 pad 5: VBUS -> (no net)
- J2 pad 6: LDO -> (no net)
- J3 pad 1: 3V3_Buck_1 -> (no net)
- J3 pad 2: VCC -> (no net)
- J3 pad 3: 3V3_Buck_2 -> (no net)
- J3 pad 4: VCC -> (no net)
- J3 pad 5: 3V3_LDO -> (no net)
- J3 pad 6: VCC -> (no net)
- R1 pad 2: Net-(J1-Pad6) -> Net-(R1-Pad2)
- R2 pad 1: LDO -> Net-(C1-Pad1)
- R2 pad 2: Net-(IC3-Pad5) -> Net-(IC1-Pad1)
- R3 pad 1: D0+ -> Net-(R1-Pad2)
- R3 pad 2: Net-(IC1-Pad2) -> Net-(IC1-Pad1)
Routing:
- net GND: track 151.4 -> 0.00 mm, vias 71 -> 0
- net VBUS: track 143.3 -> 0.00 mm, vias 5 -> 0
- net OUT2: track 92.8 -> 0.00 mm, vias 2 -> 0
- net D_DS_1_+: track 85.6 -> 0.00 mm, vias 4 -> 0
- net D_DS_1_-: track 83.8 -> 0.00 mm, vias 4 -> 0
- net D_DS_2_-: track 76.7 -> 0.00 mm, vias 3 -> 0
- net D_DS_2_+: track 74.8 -> 0.00 mm, vias 3 -> 0
- net OUT1: track 69.8 -> 0.00 mm, vias 2 -> 0
- net 3V3_Buck_1: track 67.0 -> 0.00 mm, vias 1 -> 0
- net D_DS_3_-: track 61.8 -> 0.00 mm, vias 2 -> 0
- net D_DS_3_+: track 61.8 -> 0.00 mm, vias 2 -> 0
- net 3V3_Buck_2: track 59.6 -> 0.00 mm, vias 3 -> 0
- net LDO: track 50.6 -> 0.00 mm
- net D_DS_4_-: track 48.7 -> 0.00 mm, vias 2 -> 0
- net D_DS_4_+: track 47.6 -> 0.00 mm, vias 2 -> 0
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- removed copper zone on F.Cu, net 3V3_Buck_1
- removed copper zone on F.Cu, net GND
- removed copper zone on In1.Cu, net GND
- removed copper zone on F.Cu, net LDO
- removed copper zone on In2.Cu, net VCC
Other:
- board size 86.4 x 94.7 mm -> 88.9 x 63.5 mm
- board text added: "USB HUB v3.3 by MK"
- board text removed: "3V3_1 3V3_2 LDO"
- board text removed: "B1 B2 LDO"
- board text removed: "USB HUB v3.2-EB by Maximilian Altrichter"

Commit message: orderd
Parts:
- added BR1: Bridge, SamacSys_Parts:SOP510P1005X330-4N, F.Cu at (91.5, 100.3)
- added BR2: Bridge, SamacSys_Parts:SOP510P1005X330-4N, F.Cu at (107.2, 112.0)
- added BR3: Bridge, SamacSys_Parts:SOP510P1005X330-4N, F.Cu at (107.2, 88.7)
- added BR4: Bridge, SamacSys_Parts:SOP510P1005X330-4N, F.Cu at (32.5, 88.7)
- added BR5: Bridge, SamacSys_Parts:SOP510P1005X330-4N, F.Cu at (32.5, 112.0)
- added C10: 18pF, Capacitor_SMD:C_0603_1608Metric, F.Cu at (77.5, 96.1)
- added C11: 18pF, Capacitor_SMD:C_0603_1608Metric, F.Cu at (82.0, 98.6)
- added C12: 0.1uF, Capacitor_SMD:C_0402_1005Metric, F.Cu at (73.4, 106.3)
- added C13: 0.1uF, Capacitor_SMD:C_0402_1005Metric, F.Cu at (75.3, 108.4)
- added C14: 0.1uF, Capacitor_SMD:C_0402_1005Metric, F.Cu at (76.2, 98.2)
- added C15: 0.1uF, Capacitor_SMD:C_0402_1005Metric, F.Cu at (105.5, 95.5)
- added C16: 1nF, Capacitor_SMD:C_0603_1608Metric, F.Cu at (106.7, 102.1)
- added C17: 1nF, Capacitor_SMD:C_0603_1608Metric, F.Cu at (45.3, 96.4)
- added C18: 0.1uF, Capacitor_SMD:C_0402_1005Metric, F.Cu at (94.0, 93.7)
- added C19: 0.1uF, Capacitor_SMD:C_0402_1005Metric, F.Cu at (64.6, 99.9)
- added C20: 0.1uF, Capacitor_SMD:C_0402_1005Metric, F.Cu at (112.5, 117.6)
- added C21: 100uF, SamacSys_Parts:CAPPRD350W52D800H1300, F.Cu at (94.2, 114.0)
- added C22: 1nF, Capacitor_SMD:C_0603_1608Metric, F.Cu at (84.8, 117.1)
- added C23: 100uF, SamacSys_Parts:CAPPRD350W52D800H1300, F.Cu at (49.0, 86.4)
- added C24: 1nF, Capacitor_SMD:C_0603_1608Metric, F.Cu at (55.0, 83.4)
- added C25: 0.1uF, Capacitor_SMD:C_0402_1005Metric, F.Cu at (38.9, 89.5)
- added C26: 100uF, SamacSys_Parts:CAPPRD350W52D800H1300, F.Cu at (97.5, 86.4)
- added C27: 100uF, SamacSys_Parts:CAPPRD350W52D800H1300, F.Cu at (45.5, 114.0)
- added C28: 1nF, Capacitor_SMD:C_0603_1608Metric, F.Cu at (84.8, 83.4)
- added C29: 0.1uF, Capacitor_SMD:C_0402_1005Metric, F.Cu at (112.1, 93.9)
- added C30: 1nF, Capacitor_SMD:C_0603_1608Metric, F.Cu at (55.0, 117.2)
- added C31: 0.1uF, Capacitor_SMD:C_0402_1005Metric, F.Cu at (38.9, 112.9)
- added C5: 0.1uF, Capacitor_SMD:C_0402_1005Metric, F.Cu at (66.8, 97.2)
- added C6: 0.1uF, Capacitor_SMD:C_0402_1005Metric, F.Cu at (75.1, 95.6)
- added C7: 0.1uF, Capacitor_SMD:C_0402_1005Metric, F.Cu at (70.4, 106.3)
- added C8: 0.1uF, Capacitor_SMD:C_0402_1005Metric, F.Cu at (64.7, 101.0)
- added C9: 4.7uF, Capacitor_SMD:C_1206_3216Metric, F.Cu at (63.3, 102.7)
- added D3: PWR2, LED_SMD:LED_0402_1005Metric, F.Cu at (84.3, 76.0)
- added D4: PWR3, LED_SMD:LED_0402_1005Metric, F.Cu at (55.4, 76.0)
- added D5: PWR4, LED_SMD:LED_0402_1005Metric, F.Cu at (55.4, 124.7)
- added R10: 100K, Resistor_SMD:R_0402_1005Metric, F.Cu at (69.3, 106.3)
- added R11: 100K, Resistor_SMD:R_0402_1005Metric, F.Cu at (71.4, 106.3)
- added R12: 4.7K, Resistor_SMD:R_1206_3216Metric, F.Cu at (84.4, 121.2)
- added R13: 4.7K, Resistor_SMD:R_1206_3216Metric, F.Cu at (84.4, 79.5)
- added R14: 4.7K, Resistor_SMD:R_1206_3216Metric, F.Cu at (55.4, 79.5)
- added R15: 4.7K, Resistor_SMD:R_1206_3216Metric, F.Cu at (55.4, 121.2)
- added R4: 100K, Resistor_SMD:R_0402_1005Metric, F.Cu at (74.9, 105.5)
- added R5: 100K, Resistor_SMD:R_1206_3216Metric, F.Cu at (80.9, 106.1)
- added R6: 100K, Resistor_SMD:R_0402_1005Metric, F.Cu at (74.9, 104.5)
- added R7: 100K, Resistor_SMD:R_0402_1005Metric, F.Cu at (76.2, 95.9)
- added R8: 330, Resistor_SMD:R_0603_1608Metric, F.Cu at (108.1, 95.2)
- added R9: 100K, Resistor_SMD:R_0402_1005Metric, F.Cu at (72.4, 106.3)
- added U1: USB2514B_Bi, Package_DFN_QFN:QFN-36-1EP_6x6mm_P0.5mm_EP3.7x3.7mm, F.Cu at (71.5, 100.3)
- added Y1: 24MHz 10ppm, Crystal:Crystal_SMD_2016-4Pin_2.0x1.6mm, F.Cu at (79.8, 98.8)
- C1: footprint storage:C_1uF -> Capacitor_SMD:C_0805_2012Metric
- C2: value 10uF -> 2.2uF; footprint storage:C_10uF -> Capacitor_SMD:C_0603_1608Metric
- C3, C4: footprint storage:C_0.1uF -> Capacitor_SMD:C_0402_1005Metric
- D1: value 1N4002 -> PWR; footprint storage:D_1N4002 -> LED_SMD:LED_0402_1005Metric
- D2: value 1N4002 -> PWR1; footprint storage:D_1N4002 -> LED_SMD:LED_0402_1005Metric
- IC1: value LM317MDCY -> TLV76733DGNR; footprint SamacSys_Parts:SOT230P700X180-4N -> SamacSys_Parts:SOP65P490X110-9N
- IC2: value TUSB8041IPAPRQ1 -> TPS2044BDR; footprint SamacSys_Parts:QFP50P1200X1200X120-65N -> SamacSys_Parts:SOIC127P600X175-16N
- J1: value 692221030100 -> USB_B_Micro; footprint SamacSys_Parts:WR-COM_USB_TYPE_B -> Connector_USB:USB_Micro-B_Molex-105017-0001
- J2, J3, J4, J5: value 692121030100 -> 67643-0910; footprint SamacSys_Parts:692121030100 -> SamacSys_Parts:676430910
- R1: value 22 -> 100K; footprint storage:R_22 -> Resistor_SMD:R_0402_1005Metric
- R2: value 240 -> 4.7K; footprint storage:R_240 -> Resistor_SMD:R_1206_3216Metric
- R3: value 390 -> 1Meg; footprint storage:R_390 -> Resistor_SMD:R_0805_2012Metric
- moved J5 82.2 mm to (40.5, 122.0), turned to 0 degrees
- moved J2 58.4 mm to (92.2, 122.0), turned to 0 degrees
- moved J3 49.8 mm to (99.2, 78.7)
- moved C1 40.2 mm to (110.1, 106.3)
- moved J4 39.4 mm to (47.5, 78.7)
- moved C3 31.4 mm to (71.2, 94.1), turned to 90 degrees
- moved R3 28.7 mm to (81.2, 96.0), turned to 180 degrees
- moved C2 28.5 mm to (100.2, 106.4), turned to 270 degrees
- moved C4 28.5 mm to (76.3, 102.0)
- moved J1 24.4 mm to (111.5, 100.3), turned to 90 degrees
- moved IC1 23.0 mm to (104.9, 104.9), turned to 180 degrees
- moved R2 20.8 mm to (78.4, 106.1), turned to 270 degrees
- moved D2 19.9 mm to (84.4, 124.7), turned to 90 degrees
- moved R1 16.8 mm to (74.9, 106.7)
- moved D1 14.2 mm to (78.7, 110.9), turned to 180 degrees
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Connections:
- C1 pad 1: Net-(C1-Pad1) -> +5V
- C2 pad 1: Net-(C2-Pad1) -> +3V3
- C3 pad 1: Net-(C2-Pad1) -> +3V3
- C4 pad 1: Net-(C4-Pad1) -> +3V3
- D1 pad 1: Net-(C4-Pad1) -> GND
- D1 pad 2: Net-(C1-Pad1) -> Net-(D1-Pad2)
- D2 pad 1: Net-(C2-Pad1) -> GND
- D2 pad 2: Net-(C4-Pad1) -> Net-(D2-Pad2)
- IC1 pad 1: Net-(IC1-Pad1) -> +5V
- IC1 pad 2: Net-(C1-Pad1) -> Net-(IC1-Pad2)
- IC1 pad 3: Net-(C2-Pad1) -> GND
- IC1 pad 4: Net-(C4-Pad1) -> Net-(IC1-Pad4)
- IC2 pad 1: (no net) -> GND
- IC2 pad 10: (no net) -> /PWR4
- IC2 pad 11: (no net) -> /PWR3
- IC2 pad 12: (no net) -> /OCS_N3
- IC2 pad 13: (no net) -> /OCS_N2
- IC2 pad 14: (no net) -> /PWR2
- IC2 pad 15: (no net) -> /PWR1
- IC2 pad 16: (no net) -> /OCS_N1
- IC2 pad 2: (no net) -> +5V
- IC2 pad 3: (no net) -> /PRTPWR1
- IC2 pad 4: (no net) -> /PRTPWR2
- IC2 pad 5: (no net) -> GND
- IC2 pad 6: (no net) -> +5V
- IC2 pad 7: (no net) -> /PRTPWR3
- IC2 pad 8: (no net) -> /PRTPWR4
- IC2 pad 9: (no net) -> /OCS_N4
- J1 pad 1: (no net) -> +5V
- J1 pad 2: (no net) -> /USBUP_-
- J1 pad 3: (no net) -> /USBUP_+
- J1 pad 4: (no net) -> Net-(J1-Pad4)
- J1 pad 5: (no net) -> Net-(C15-Pad2)
- J1 pad 6: (no net) -> Net-(C15-Pad2)
- J2 pad 1: (no net) -> /PWR1
- J2 pad 2: (no net) -> /USBDN_1-
- J2 pad 3: (no net) -> /USBDN_1+
- J2 pad 4: (no net) -> GND
- J3 pad 1: (no net) -> /PWR2
- J3 pad 2: (no net) -> /USBDN_2-
- J3 pad 3: (no net) -> /USBDN_2+
- J3 pad 4: (no net) -> GND
- J4 pad 1: (no net) -> /PWR3
- J4 pad 2: (no net) -> /USBDN_3-
- J4 pad 3: (no net) -> /USBDN_3+
- J4 pad 4: (no net) -> GND
- J5 pad 1: (no net) -> /PWR4
- J5 pad 2: (no net) -> /USBDN_4-
- J5 pad 3: (no net) -> /USBDN_4+
- J5 pad 4: (no net) -> GND
- R1 pad 1: GND -> Net-(C12-Pad1)
- R1 pad 2: Net-(R1-Pad2) -> +3V3
- R2 pad 1: Net-(C1-Pad1) -> /LOCAL_PWR
- R2 pad 2: Net-(IC1-Pad1) -> Net-(D1-Pad2)
- R3 pad 1: Net-(R1-Pad2) -> /XTALOUT
- R3 pad 2: Net-(IC1-Pad1) -> /XTALIN
Routing:
- net GND: track 0.00 -> 131.0 mm, vias 0 -> 71
- net +5V: track 0.00 -> 120.1 mm, vias 0 -> 6
- net /PWR1: track 0.00 -> 91.0 mm, vias 0 -> 8
- net /PWR2: track 0.00 -> 88.8 mm, vias 0 -> 4
- net /USBDN_1+: track 0.00 -> 65.3 mm, vias 0 -> 2
- net /USBDN_4+: track 0.00 -> 65.2 mm
- net /USBDN_3-: track 0.00 -> 63.9 mm, vias 0 -> 2
- net /USBDN_1-: track 0.00 -> 62.0 mm, vias 0 -> 2
- net /USBDN_4-: track 0.00 -> 61.7 mm, vias 0 -> 2
- net /USBDN_3+: track 0.00 -> 54.0 mm
- net /USBDN_2+: track 0.00 -> 50.5 mm
- net /PWR4: track 0.00 -> 49.7 mm, vias 0 -> 2
- net /PWR3: track 0.00 -> 49.5 mm, vias 0 -> 2
- net /USBDN_2-: track 0.00 -> 49.1 mm
- net /USBUP_+: track 0.00 -> 46.2 mm, vias 0 -> 2
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- added copper zone on In2.Cu, net +3V3
- added copper zone on F.Cu, net GND
- added copper zone on In1.Cu, net GND
