File: USB_HUB.sch (KiCad schematic (older format))
At the start: 21 parts, among them J1 USB_PORT_1, J2 USB_Port_2, J3 USB_Port_3, J4 USB_Port_4, U1 FE1.1s, Y1 X322512MSB4SI

Commit message: added atmega32 schematic
Parts:
- removed R5: 1K, Resistor_SMD:R_0603_1608Metric, symbol Device:R_Small
- removed Y1: X322512MSB4SI, crystal_12MHz:X322512MSB4SI, symbol X322512MSB4SI:X322512MSB4SI
- added R1: 1.5K, Resistor_SMD:R_0603_1608Metric, symbol Device:R_Small
- added Y1: X322512MSB4SI, max_KiCAD_lib:X322512MSB4SI, symbol max_KiCAD_lib:X322512MSB4SI
- R3, R4: value 1K -> 1.5K
Other:
- moved on the sheet: C1, C2, C3, C4, C5, C6, D1, D2, D3, D4, D5, J1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

Commit message: file: finished schematic
Changed lines of the file:
@@
 	0    1    1    0
 $EndComp
+Text HLabel 6100 4350 2    50   Output ~ 0
+D4_P
+Text HLabel 6100 4450 2    50   Output ~ 0
+D4_N
 $EndSCHEMATC

Commit message: pcb schematic and layout edit i.e. finished -> orderd pcb jlcpcb
Parts:
- C1, C3, C5: LCSC Part # (none) -> C15850
- C2, C4, C6: LCSC Part # (none) -> C14663
- D1, D2, D3, D4: LCSC Part # (none) -> C72041
- D5: LCSC Part # (none) -> C2297
- J1: value USB_PORT_1 -> USB_Port_1; LCSC Part # (none) -> C163037
- J2, J3, J4: LCSC Part # (none) -> C163037
- R1, R3, R4: LCSC Part # (none) -> C22843
- R2: LCSC Part # (none) -> C13167
- Y1: LCSC Part # (none) -> C9002
Connections:
- net D1_N: now also J4.3 (Pin_3); no longer J1.4 (Pin_4)
- net D1_P: now also J4.4 (Pin_4); no longer J1.3 (Pin_3)
- net D2_N: now also J3.3 (Pin_3); no longer J2.4 (Pin_4)
- net D2_P: now also J3.4 (Pin_4); no longer J2.3 (Pin_3)
- net D3_N: now also J2.3 (Pin_3); no longer J3.4 (Pin_4)
- net D3_P: now also J2.4 (Pin_4); no longer J3.3 (Pin_3)
- net D4_N: now also J1.3 (Pin_3); no longer J4.4 (Pin_4)
- net D4_P: now also J1.4 (Pin_4); no longer J4.3 (Pin_3)
- net DRV: now also D1.2 (A), D2.1 (K), D3.2 (A), D4.1 (K); no longer D1.1 (K), D2.2 (A), D3.1 (K), D4.2 (A)
- new net: D1.1 (K), D2.2 (A), R4.1
- new net: D3.1 (K), D4.2 (A), R1.1
- no-connect marks 4 -> 6
Other:
- moved on the sheet: D1, D2, D3, D4
Changed lines of the file:
@@
 DRV
-$Comp
-L Device:LED_Small D1
-U 1 1 61289E27
-P 7350 4750
-F 0 "D1" H 7450 4800 50  0000 C CNN
-F 1 "Port_1" H 7200 4800 50  0000 C CNN
-F 2 "LED_SMD:LED_0603_1608Metric" V 7350 4750 50  0001 C CNN
-F 3 "~" V 7350 4750 50  0001 C CNN
-	1    7350 4750
-	-1   0    0    1
-$EndComp
 $Comp
 L Device:LED_Small D5
@@
 F 2 "LED_SMD:LED_0805_2012Metric_Castellated" V 8050 4750 50  0001 C CNN
 F 3 "~" V 8050 4750 50  0001 C CNN
+F 4 "C2297" H 8050 4750 50  0001 C CNN "LCSC Part #"
 	1    8050 4750
 	-1   0    0    1
@@
 Text Label 6100 4950 2    50   ~ 0
 LED2
-$Comp
-L Device:LED_Small D2
-U 1 1 61290640
-P 7350 4950
-F 0 "D2" H 7250 5000 50  0000 C CNN
-F 1 "Port_3" H 7500 4900 50  0000 C CNN
-F 2 "LED_SMD:LED_0603_1608Metric" V 7350 4950 50  0001 C CNN
-F 3 "~" V 7350 4950 50  0001 C CNN
-	1    7350 4950
-	1    0    0    -1
-$EndComp
 Wire Wire Line
 	7250 4750 7150 4750
@@
 F 2 "Resistor_SMD:R_0603_1608Metric" H 7000 5200 50  0001 C CNN
 F 3 "~" H 7000 5200 50  0001 C CNN
+F 4 "C22843" H 7000 5200 50  0001 C CNN "LCSC Part #"
 	1    7000 5200
 	0    1    1    0
-$EndComp
-$Comp
-L Device:LED_Small D3
-U 1 1 61294F3C
-P 7350 5100
-F 0 "D3" H 7450 5150 50  0000 C CNN
-F 1 "Port_2" H 7200 5150 50  0000 C CNN
-F 2 "LED_SMD:LED_0603_1608Metric" V 7350 5100 50  0001 C CNN
-F 3 "~" V 7350 5100 50  0001 C CNN
-	1    7350 5100
-	-1   0    0    1
-$EndComp
-$Comp
-L Device:LED_Small D4
-U 1 1 61294F42
-P 7350 5300
-F 0 "D4" H 7250 5350 50  0000 C CNN
-F 1 "Port_4" H 7500 5250 50  0000 C CNN
-F 2 "LED_SMD:LED_0603_1608Metric" V 7350 5300 50  0001 C CNN
-F 3 "~" V 7350 5300 50  0001 C CNN
-	1    7350 5300
-	1    0    0    -1
 $EndComp
 Wire Wire Line
@@
 F 2 "Resistor_SMD:R_0603_1608Metric" H 4200 5250 50  0001 C CNN
 F 3 "~" H 4200 5250 50  0001 C CNN
+F 4 "C13167" H 4200 5250 50  0001 C CNN "LCSC Part #"
 	1    4200 5250
 	0    1    1    0
@@
 F 2 "Capacitor_SMD:C_0603_1608Metric" H 6150 2200 50  0001 C CNN
 F 3 "~" H 6150 2200 50  0001 C CNN
+F 4 "C14663" H 6150 2200 50  0001 C CNN "LCSC Part #"
 	1    6150 2200
 	1    0    0    -1
@@
 F 2 "Capacitor_SMD:C_0805_2012Metric" H 5800 2200 50  0001 C CNN
 F 3 "~" H 5800 2200 50  0001 C CNN
+F 4 "C15850" H 5800 2200 50  0001 C CNN "LCSC Part #"
 	1    5800 2200
 	1    0    0    -1
@@
 F 2 "Capacitor_SMD:C_0603_1608Metric" H 4550 2200 50  0001 C CNN
 F 3 "~" H 4550 2200 50  0001 C CNN
+F 4 "C14663" H 4550 2200 50  0001 C CNN "LCSC Part #"
 	1    4550 2200
 	1    0    0    -1
@@
 F 2 "Capacitor_SMD:C_0805_2012Metric" H 4200 2200 50  0001 C CNN
 F 3 "~" H 4200 2200 50  0001 C CNN
+F 4 "C15850" H 4200 2200 50  0001 C CNN "LCSC Part #"
 	1    4200 2200
 	1    0    0    -1
@@
 F 2 "Capacitor_SMD:C_0603_1608Metric" H 5350 2200 50  0001 C CNN
 F 3 "~" H 5350 2200 50  0001 C CNN
+F 4 "C14663" H 5350 2200 50  0001 C CNN "LCSC Part #"
 	1    5350 2200
 	1    0    0    -1
@@
 F 2 "Capacitor_SMD:C_0805_2012Metric" H 5000 2200 50  0001 C CNN
 F 3 "~" H 5000 2200 50  0001 C CNN
+F 4 "C15850" H 5000 2200 50  0001 C CNN "LCSC Part #"
 	1    5000 2200
 	1    0    0    -1
@@
 P 10350 3600
 F 0 "J1" H 10378 3576 50  0000 L CNN
-F 1 "USB_PORT_1" H 10378 3485 50  0000 L CNN
+F 1 "USB_Port_1" H 10378 3485 50  0000 L CNN
 F 2 "Connector_JST:JST_XH_S4B-XH-A-1_1x04_P2.50mm_Horizontal" H 10350 3600 50  0001 C CNN
 F 3 "~" H 10350 3600 50  0001 C CNN
+F 4 "C163037" H 10350 3600 50  0001 C CNN "LCSC Part #"
 	1    10350 3600
 	1    0    0    -1
@@
 F 2 "Connector_JST:JST_XH_S4B-XH-A-1_1x04_P2.50mm_Horizontal" H 10350 4100 50  0001 C CNN
 F 3 "~" H 10350 4100 50  0001 C CNN
+F 4 "C163037" H 10350 4100 50  0001 C CNN "LCSC Part #"
 	1    10350 4100
 	1    0    0    -1
@@
 F 2 "Connector_JST:JST_XH_S4B-XH-A-1_1x04_P2.50mm_Horizontal" H 10350 4600 50  0001 C CNN
 F 3 "~" H 10350 4600 50  0001 C CNN
+F 4 "C163037" H 10350 4600 50  0001 C CNN "LCSC Part #"
 	1    10350 4600
 	1    0    0    -1
@@
 F 2 "Connector_JST:JST_XH_S4B-XH-A-1_1x04_P2.50mm_Horizontal" H 10350 5100 50  0001 C CNN
 F 3 "~" H 10350 5100 50  0001 C CNN
+F 4 "C163037" H 10350 5100 50  0001 C CNN "LCSC Part #"
 	1    10350 5100
 	1    0    0    -1
@@
 	10150 3600 9850 3600
 Wire Wire Line
+	10150 5200 9850 5200
+Wire Wire Line
+	10150 5300 9850 5300
+Wire Wire Line
+	10150 4000 9850 4000
+Wire Wire Line
+	10150 4100 9850 4100
+Wire Wire Line
+	10150 4700 9850 4700
+Wire Wire Line
+	10150 4800 9850 4800
+Wire Wire Line
+	10150 4500 9850 4500
+Wire Wire Line
+	10150 4600 9850 4600
+Wire Wire Line
+	10150 4200 9850 4200
+Wire Wire Line
+	10150 4300 9850 4300
+Wire Wire Line
+	10150 5000 9850 5000
+Wire Wire Line
+	10150 5100 9850 5100
+Wire Wire Line
 	10150 3700 9850 3700
 Wire Wire Line
 	10150 3800 9850 3800
-Wire Wire Line
-	10150 4000 9850 4000
-Wire Wire Line
-	10150 4100 9850 4100
-Wire Wire Line
-	10150 4200 9850 4200
-Wire Wire Line
-	10150 4300 9850 4300
-Wire Wire Line
-	10150 4500 9850 4500
-Wire Wire Line
-	10150 4600 9850 4600
-Wire Wire Line
-	10150 4700 9850 4700
-Wire Wire Line
-	10150 4800 9850 4800
-Wire Wire Line
-	10150 5000 9850 5000
-Wire Wire Line
-	10150 5100 9850 5100
-Wire Wire Line
-	10150 5200 9850 5200
-Wire Wire Line
-	10150 5300 9850 5300
 $Comp
 L power:+5V #PWR0115
@@
 	0    1    1    0
 $EndComp
+Text Label 9850 5300 0    50   ~ 0
+D1_P
+Text Label 9850 5200 0    50   ~ 0
+D1_N
+Text Label 9850 4800 0    50   ~ 0
+D2_P
+Text Label 9850 4300 0    50   ~ 0
+D3_P
+Text Label 9850 3800 0    50   ~ 0
+D4_P
+Text Label 9850 4700 0    50   ~ 0
+D2_N
+Text Label 9850 4200 0    50   ~ 0
+D3_N
 Text Label 9850 3700 0    50   ~ 0
-D1_P
-Text Label 9850 3800 0    50   ~ 0
-D1_N
-Text Label 9850 4200 0    50   ~ 0
-D2_P
-Text Label 9850 4700 0    50   ~ 0
-D3_P
-Text Label 9850 5200 0    50   ~ 0
-D4_P
-Text Label 9850 4300 0    50   ~ 0
-D2_N
-Text Label 9850 4800 0    50   ~ 0
-D3_N
-Text Label 9850 5300 0    50   ~ 0
 D4_N
 $Comp
@@
 F 6 "Yangxing Tech" H 3200 4750 50  0001 L CNN "Manufacturer_Name"
 F 7 "X322512MSB4SI" H 3200 4650 50  0001 L CNN "Manufacturer_Part_Number"
+F 8 "C9002" H 1750 5050 50  0001 C CNN "LCSC Part #"
 	1    1750 5050
 	1    0    0    -1
@@
 F 2 "Resistor_SMD:R_0603_1608Metric" H 7000 4850 50  0001 C CNN
 F 3 "~" H 7000 4850 50  0001 C CNN
+F 4 "C22843" H 7000 4850 50  0001 C CNN "LCSC Part #"
 	1    7000 4850
 	0    1    1    0
@@
 F 2 "Resistor_SMD:R_0603_1608Metric" H 8350 4750 50  0001 C CNN
 F 3 "~" H 8350 4750 50  0001 C CNN
+F 4 "C22843" H 8350 4750 50  0001 C CNN "LCSC Part #"
 	1    8350 4750
 	0    1    1    0
@@
 Text HLabel 6100 4450 2    50   Output ~ 0
 D4_N
+$Comp
+L Device:LED_Small D4
+U 1 1 61294F42
+P 7350 4750
+F 0 "D4" H 7250 4800 50  0000 C CNN
+F 1 "Port_4" H 7500 4700 50  0000 C CNN
+F 2 "LED_SMD:LED_0603_1608Metric" V 7350 4750 50  0001 C CNN
+F 3 "~" V 7350 4750 50  0001 C CNN
+F 4 "C72041" H 7350 4750 50  0001 C CNN "LCSC Part #"
+	1    7350 4750
+	-1   0    0    1
+$EndComp
+$Comp
+L Device:LED_Small D1
+U 1 1 61289E27
+P 7350 5300
+F 0 "D1" H 7450 5350 50  0000 C CNN
+F 1 "Port_1" H 7200 5350 50  0000 C CNN
+F 2 "LED_SMD:LED_0603_1608Metric" V 7350 5300 50  0001 C CNN
+F 3 "~" V 7350 5300 50  0001 C CNN
+F 4 "C72041" H 7350 5300 50  0001 C CNN "LCSC Part #"
+	1    7350 5300
+	1    0    0    -1
+$EndComp
+$Comp
+L Device:LED_Small D3
+U 1 1 61294F3C
+P 7350 4950
+F 0 "D3" H 7450 5000 50  0000 C CNN
+F 1 "Port_2" H 7200 5000 50  0000 C CNN
+F 2 "LED_SMD:LED_0603_1608Metric" V 7350 4950 50  0001 C CNN
+F 3 "~" V 7350 4950 50  0001 C CNN
+F 4 "C72041" H 7350 4950 50  0001 C CNN "LCSC Part #"
+	1    7350 4950
+	1    0    0    -1
+$EndComp
+$Comp
+L Device:LED_Small D2
+U 1 1 61290640
+P 7350 5100
+F 0 "D2" H 7250 5150 50  0000 C CNN
+F 1 "Port_3" H 7500 5050 50  0000 C CNN
+F 2 "LED_SMD:LED_0603_1608Metric" V 7350 5100 50  0001 C CNN
+F 3 "~" V 7350 5100 50  0001 C CNN
+F 4 "C72041" H 7350 5100 50  0001 C CNN "LCSC Part #"
+	1    7350 5100
+	-1   0    0    1
+$EndComp
+NoConn ~ 2400 800
+NoConn ~ -4850 150
 $EndSCHEMATC
